File: UccMicroDuino/UccMicroDuino.kicad_pcb (KiCad board)
At the start: 2 copper layers, 45 x 45 mm, 14 parts, among them J1 Pcb USB Type A, J2 Header, U1 ATtiny85-20SU

Commit message: Mi primer versionado con gitbush (Modificado)
Routing:
- net Net-(D2-K): track 28.2 -> 30.2 mm
- net Net-(D3-K): track 40.1 -> 41.7 mm
- net GND: track 121.2 -> 122.6 mm
Changed lines of the file:
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@@
 	)
 	(segment
-		(start 177 106.5)
-		(end 179 106.5)
+		(start 183.399 102.101)
+		(end 181.5 104)
 		(width 0.6)
 		(layer "F.Cu")
@@
 	)
 	(segment
-		(start 179 106.5)
-		(end 183.399 102.101)
+		(start 181.5 106.5)
+		(end 177 106.5)
 		(width 0.6)
 		(layer "F.Cu")
@@
 	)
 	(segment
+		(start 181.5 104)
+		(end 181.5 106.5)
+		(width 0.6)
+		(layer "F.Cu")
+		(net 1)
+	)
+	(segment
 		(start 215.252 84.522852)
 		(end 206.427147 75.698)
@@
 	)
 	(segment
-		(start 183.5 108.85)
-		(end 183.5 105.5)
-		(width 0.6)
-		(layer "F.Cu")
-		(net 4)
-	)
-	(segment
 		(start 188 104.35)
 		(end 186.5 102.85)
@@
 	)
 	(segment
-		(start 183.5 105.5)
-		(end 184 105.5)
+		(start 184 105.5)
+		(end 184 111)
+		(width 0.6)
+		(layer "F.Cu")
+		(net 4)
+	)
+	(segment
+		(start 184 111)
+		(end 177.5 111)
 		(width 0.6)
 		(layer "F.Cu")
@@
 	)
 	(segment
-		(start 177.5 111)
-		(end 181.35 111)
-		(width 0.6)
-		(layer "F.Cu")
-		(net 4)
-	)
-	(segment
 		(start 186.5 97.5)
 		(end 186.5 92)
@@
 	)
 	(segment
-		(start 181.35 111)
-		(end 183.5 108.85)
+		(start 184 111)
+		(end 184.5 111.5)
 		(width 0.6)
 		(layer "F.Cu")
@@
 	)
 	(segment
-		(start 180.25 109)
-		(end 181.75 107.5)
+		(start 182.899 105.043951)
+		(end 182.899 109)
+		(width 0.6)
+		(layer "F.Cu")
+		(net 5)
+	)
+	(segment
+		(start 184.5 103.442951)
+		(end 182.899 105.043951)
 		(width 0.6)
 		(layer "F.Cu")
@@
 	)
 	(segment
-		(start 177.5 109)
-		(end 180.25 109)
-		(width 0.6)
-		(layer "F.Cu")
-		(net 5)
-	)
-	(segment
 		(start 184.442951 103)
 		(end 184.5 103)
@@
 	)
 	(segment
-		(start 181.75 105.692951)
-		(end 184.442951 103)
+		(start 182.899 109)
+		(end 177.5 109)
 		(width 0.6)
 		(layer "F.Cu")
@@
 	)
 	(segment
-		(start 181.75 107.5)
-		(end 181.75 105.692951)
-		(width 0.6)
-		(layer "F.Cu")
+		(start 184.5 103)
+		(end 184.5 103.442951)
+		(width 0.6)
+		(layer "F.Cu")
